File: rpi-fan-ctl.kicad_pcb (KiCad board)
At the start: 4 copper layers, 37.3 x 25.4 mm, 27 parts, among them U1 74LVC2G17, U2 74LVC2G17

Commit message: finish?
Parts:
- added G***: LOGO, LOGO, B.Cu at (99.5, 62.5)
- moved C1 69.5 mm to (104.8, 66.1)
- moved D2 69.5 mm to (99.0, 58.5)
- moved D4 69.5 mm to (107.4, 66.1)
- moved R3 69.5 mm to (87.2, 66.1)
- moved R4 69.5 mm to (99.0, 61.0)
- moved R8 69.5 mm to (100.3, 64.8)
- moved C2 69.5 mm to (104.8, 53.4)
- moved C3 69.5 mm to (93.0, 71.2)
- moved C4 69.5 mm to (93.0, 63.6)
- moved D1 69.5 mm to (107.4, 53.3)
- moved D3 69.5 mm to (87.2, 61.0)
- moved D5 69.5 mm to (104.8, 58.5)
- moved D6 69.5 mm to (104.8, 71.2)
- moved FAN1 69.5 mm to (112.5, 52.1)
- moved FAN2 69.5 mm to (112.5, 64.8)
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Routing:
- net +5V: track 0.00 -> 82.0 mm, vias 0 -> 6
- net GND: track 0.00 -> 25.4 mm, vias 0 -> 46
- net +3.3V: track 5.34 -> 17.8 mm, vias 0 -> 1
- net TACH2_5V: track 22.3 -> 18.4 mm
- net TACH1_3V3: track 32.7 -> 30.2 mm
- net TACH2_3V3: track 25.4 -> 24.3 mm
- net PWM_CTL_5V: track 44.4 -> 45.4 mm
- added copper zone on B.Cu, net GND
- added copper zone on F.Cu, net GND
Other:
- board size 37.3 x 25.4 mm -> 37.8 x 25 mm
- board text added: "PWM"
- board text added: "rPi_fan_ctl v0.1.0"
- board text added: "regensberry"
- board text removed: "rPi_FAN_CTL v1.0.0"

Commit message: made all preview connectors angled
Parts:
- RPI1: footprint Connector_PinHeader_2.54mm:PinHeader_1x05_P2.54mm_Vertical -> Connector_PinHeader_2.54mm:PinHeader_1x05_P2.54mm_Horizontal
- moved RPI1 10.2 mm to (82.6, 71.2), turned to 180 degrees
Connections:
- R1 pad 1: Net-(RPI1-Pin_5) -> Net-(RPI1-Pin_1)
- R2 pad 1: Net-(RPI1-Pin_4) -> Net-(RPI1-Pin_2)
- RPI1 pad 1: GND -> Net-(RPI1-Pin_1)
- RPI1 pad 2: +3.3V -> Net-(RPI1-Pin_2)
- RPI1 pad 4: Net-(RPI1-Pin_4) -> +3.3V
- RPI1 pad 5: Net-(RPI1-Pin_5) -> GND
Routing:
- net Net-(RPI1-Pin_5): track 3.47 -> 0.00 mm
- net Net-(RPI1-Pin_4): track 3.47 -> 0.00 mm
- net Net-(RPI1-Pin_2): track 0.00 -> 3.47 mm
- net Net-(RPI1-Pin_1): track 0.00 -> 3.47 mm
Other:
- board text added: "rPi_fan_ctl v0.1.1 01/25"
- board text removed: "rPi_fan_ctl v0.1.0"

Commit message: updated voltage level converter
Parts:
- moved G*** 48.8 mm to (148.2, 62.5)
Changed lines of the file:
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@@
 	(footprint "LOGO"
 		(layer "B.Cu")
-		(at 99.5 62.502658 180)
+		(at 148.25 62.5 180)
 		(property "Reference" "G***"
 			(at 0 0 0)
@@
 	)
 	(gr_text "regensberry"
-		(at 86.5 62.5 270)
+		(at 135.25 62.5 270)
 		(layer "B.SilkS")
 		(effects
