File: fanctl.kicad_sch (KiCad schematic)
At the start: 28 parts, among them U1 SN74HCT125DR, U2 SN74HCT125DR

Commit message: WIP preview sch
Parts:
- added D8: LTST-C191TBKT, Diode_SMD:D_0402_1005Metric_Pad0.77x0.64mm_HandSolder, symbol J-Link-SWD-rescue:LTST-C191TBKT-dk_LED-Indication-Discrete
- added J1: Raspberry_Pi_4, Connector_PinSocket_2.54mm:PinSocket_2x21_P2.54mm_Horizontal, symbol Connector:Raspberry_Pi_4
- added J2: Conn_01x40, symbol Connector_Generic:Conn_01x40
- added R14, R15, R18, R19: 0R, Resistor_SMD:R_0603_1608Metric_Pad0.98x0.95mm_HandSolder, symbol Device:R
- added R16: 1K, Resistor_SMD:R_0603_1608Metric_Pad0.98x0.95mm_HandSolder, symbol Device:R
Connections:
- net +3.3V: now also J1.1 (3V3), J1.17 (3V3); no longer U1.4, U1.5
- net +5V: now also J1.2 (5V), J1.4 (5V)
- net GND: now also U1.4, D8.2, J1.14 (GND), J1.20 (GND), J1.25 (GND), J1.30 (GND), J1.34 (GND), J1.39 (GND), J1.6 (GND), J1.9 (GND)
- net PWM_CTL_3V3: no longer R13.2, U1.2
- net TACH1_3V3: now also R19.1
- net TACH2_3V3: now also R18.1
- net at U1.6: now also R16.1
- new net: J1.32 (GPIO12/PWM0), R15.2
- new net: J1.33 (GPIO13/PWM1), R14.2
- new net: D8.1, R16.2
- new net: J1.10 (GPIO15/UART_RXD), R18.2
- new net: J1.8 (GPIO14/UART_TXD), R19.2
- new net PWM0_3V3: R15.1, U1.5
- new net PWM_FAN_CTL_3V3: R13.2, R14.1, U1.2
Other:
- moved on the sheet: D2, D5, D6, R4, R6, R9, U1B

Commit message: release candidate
Parts:
- removed J2: Conn_01x40, symbol Connector_Generic:Conn_01x40
- removed R1, R2, R3: 0R, Resistor_SMD:R_0603_1608Metric_Pad0.98x0.95mm_HandSolder, symbol Device:R
- removed RPI1: Conn_01x05, Connector_PinHeader_2.54mm:PinHeader_1x05_P2.54mm_Horizontal, symbol Connector_Generic:Conn_01x05
- removed SUP1: Conn_01x02, Connector_PinHeader_2.54mm:PinHeader_1x02_P2.54mm_Horizontal, symbol Connector_Generic:Conn_01x02
- added J4: Raspberry_Pi_4, Connector_PinHeader_2.54mm:PinHeader_2x20_P2.54mm_Vertical, symbol Connector:Raspberry_Pi_4
- C1, C2: footprint Capacitor_SMD:C_0603_1608Metric_Pad1.08x0.95mm_HandSolder -> Capacitor_SMD:C_0805_2012Metric_Pad1.18x1.45mm_HandSolder
- J1: footprint Connector_PinSocket_2.54mm:PinSocket_2x21_P2.54mm_Horizontal -> Connector_PinSocket_2.54mm:PinSocket_2x20_P2.54mm_Horizontal
Connections:
- net +3.3V: now also J4.1 (3V3), J4.17 (3V3)
- net +5V: now also J4.2 (5V), J4.4 (5V)
- net GND: now also J4.14 (GND), J4.20 (GND), J4.25 (GND), J4.30 (GND), J4.34 (GND), J4.39 (GND), J4.6 (GND), J4.9 (GND)
- net at J1.32 (GPIO12/PWM0), R15.2: now also J4.32 (GPIO12/PWM0)
- net at J1.33 (GPIO13/PWM1), R14.2: now also J4.33 (GPIO13/PWM1)
- net at J1.10 (GPIO15/UART_RXD), R18.2: now also J4.10 (GPIO15/UART_RXD)
- net at J1.11 (GPIO17/SPI1_~{CE1}): now also J4.11 (GPIO17/SPI1_~{CE1})
- net at J1.12 (GPIO18/SPI1_~{CE0}/PCM_CLK/PWM0): now also J4.12 (GPIO18/SPI1_~{CE0}/PCM_CLK/PWM0)
- net at J1.13 (GPIO27/SDIO_DAT3): now also J4.13 (GPIO27/SDIO_DAT3)
- net at J1.15 (GPIO22/SDIO_CLK): now also J4.15 (GPIO22/SDIO_CLK)
- net at J1.16 (GPIO23/SDIO_CMD): now also J4.16 (GPIO23/SDIO_CMD)
- net at J1.18 (GPIO24/SDIO_DAT0): now also J4.18 (GPIO24/SDIO_DAT0)
- net at J1.19 (MOSI_SPI0/GPIO10): now also J4.19 (MOSI_SPI0/GPIO10)
- net at J1.21 (MISO_SPI0/GPIO09): now also J4.21 (MISO_SPI0/GPIO09)
- net at J1.22 (GPIO25/SDIO_DAT1): now also J4.22 (GPIO25/SDIO_DAT1)
- net at J1.23 (SCLK_SPI0/GPIO11): now also J4.23 (SCLK_SPI0/GPIO11)
- net at J1.24 (~{CE0}_SPI0/GPIO08): now also J4.24 (~{CE0}_SPI0/GPIO08)
- net at J1.26 (~{CE1}_SPI0/GPIO07): now also J4.26 (~{CE1}_SPI0/GPIO07)
- net at J1.27 (ID_SD_I2C0/GPIO00): now also J4.27 (ID_SD_I2C0/GPIO00)
- net at J1.28 (ID_SC_I2C0/GPIO01): now also J4.28 (ID_SC_I2C0/GPIO01)
- net at J1.29 (GPCLK1/GPIO05): now also J4.29 (GPCLK1/GPIO05)
- net at J1.3 (SDA_I2C1/GPIO02): now also J4.3 (SDA_I2C1/GPIO02)
- net at J1.31 (GPCLK2/GPIO06): now also J4.31 (GPCLK2/GPIO06)
- net at J1.35 (GPIO19/SPI1_MISO/PCM_FS): now also J4.35 (GPIO19/SPI1_MISO/PCM_FS)
- net at J1.36 (GPIO16/SPI1_~{CE2}): now also J4.36 (GPIO16/SPI1_~{CE2})
- net at J1.37 (GPIO26/SDIO_DAT2): now also J4.37 (GPIO26/SDIO_DAT2)
- net at J1.38 (GPIO20/SPI1_MOSI/PCM_DIN/PWM1): now also J4.38 (GPIO20/SPI1_MOSI/PCM_DIN/PWM1)
- net at J1.40 (GPIO21/SPI1_SCLK/PCM_DOUT): now also J4.40 (GPIO21/SPI1_SCLK/PCM_DOUT)
- net at J1.5 (SCL_I2C1/GPIO03): now also J4.5 (SCL_I2C1/GPIO03)
- net at J1.7 (GPCLK0/GPIO04): now also J4.7 (GPCLK0/GPIO04)
- net at J1.8 (GPIO14/UART_TXD), R19.2: now also J4.8 (GPIO14/UART_TXD)
Other:
- moved on the sheet: C3, C4, D2, D3, D5, D6, D8, J1, R10, R11, R13, R14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

Commit message: rotated pin headers so they are actually right
Parts:
- removed R11, R8: 33K, Resistor_SMD:R_0603_1608Metric_Pad0.98x0.95mm_HandSolder, symbol Device:R
- C1, C2: footprint Capacitor_SMD:C_0805_2012Metric_Pad1.18x1.45mm_HandSolder -> Capacitor_SMD:C_0805_2012Metric
- C3, C4: footprint Capacitor_SMD:C_0603_1608Metric_Pad1.08x0.95mm_HandSolder -> Capacitor_SMD:C_0805_2012Metric
- R10, R7: value 18K -> 10K
- R14, R15, R18, R19: value 0R -> 120R
Connections:
- net +3.3V: now also R10.1, R7.1
- net TACH1: now reaches U2.2
- net TACH1: now also FAN1.3 (Pin_3), R10.2; no longer R7.2
- net TACH2: now reaches U2.5
- net TACH2: now also FAN2.3 (Pin_3), R7.2; no longer R10.2
- removed net TACH1_5V: FAN1.3 (Pin_3), R7.1
- removed net TACH2_5V: FAN2.3 (Pin_3), R10.1
Other:
- moved on the sheet: C1, C2, D1, D4, FAN1, FAN2, R10, R13, R7, U1A, U2A, U2B
