File: fanctl.kicad_pcb (KiCad board)
At the start: 4 copper layers, 51 x 64 mm, 30 parts, among them J1 Raspberry_Pi_4, J4 Raspberry_Pi_4, U1 SN74HCT125DR, U2 SN74HCT125DR

Commit message: pcb review from @lukekaese
much thanks!
Other:
- board text added: "${TITLE} ${REVISION} 02/25 5V ONLY FANS"
- board text removed: "${TITLE} ${REVISION} 02/25 5V FANS ONLY"
Changed lines of the file:
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@@
 		(title "rPi-fanctl")
 		(date "2025-01-18")
-		(rev "v0.4.1")
+		(rev "v0.4.2")
 	)
 	(layers
@@
 		(tags "diode handsolder")
 		(property "Reference" "D2"
-			(at 2.5 0 360)
+			(at 2.5 0 0)
 			(layer "F.SilkS")
 			(effects
@@
 		(layer "Edge.Cuts")
 	)
-	(gr_text "${TITLE}\n${REVISION} 02/25\n5V FANS ONLY"
+	(gr_text "${TITLE}\n${REVISION} 02/25\n5V ONLY FANS"
 		(at 64.5 50.75 0)
 		(layer "F.SilkS")
@@
 	)
 	(via
-		(at 64.359999 91.5)
+		(at 64.359999 91.4)
 		(size 0.8)
 		(drill 0.4)
@@
 	)
 	(via
-		(at 46.579999 93.5)
+		(at 46.579999 93.6)
 		(size 0.8)
 		(drill 0.4)
@@
 	)
 	(via
-		(at 61.819999 93.5)
+		(at 61.819999 93.6)
 		(size 0.8)
 		(drill 0.4)
@@
 	)
 	(via
-		(at 77.059999 93.5)
+		(at 77.059999 93.6)
 		(size 0.8)
 		(drill 0.4)
@@
 	)
 	(via
-		(at 66.899999 93.5)
+		(at 66.899999 93.6)
 		(size 0.8)
 		(drill 0.4)
@@
 	)
 	(via
-		(at 61.819999 91.5)
+		(at 61.819999 91.4)
 		(size 0.8)
 		(drill 0.4)
@@
 	)
 	(via
-		(at 74.519999 93.5)
+		(at 74.519999 93.6)
 		(size 0.8)
 		(drill 0.4)
@@
 	)
 	(via
-		(at 46.579999 91.5)
+		(at 46.579999 91.4)
 		(size 0.8)
 		(drill 0.4)
@@
 	)
 	(via
-		(at 59.279999 93.5)
+		(at 59.279999 93.6)
 		(size 0.8)
 		(drill 0.4)
@@
 	)
 	(via
-		(at 54.199999 93.5)
+		(at 54.199999 93.6)
 		(size 0.8)
 		(drill 0.4)
@@
 	)
 	(via
-		(at 59.279999 91.5)
+		(at 59.279999 91.4)
 		(size 0.8)
 		(drill 0.4)
@@
 	)
 	(via
-		(at 51.659999 91.5)
+		(at 51.659999 91.4)
 		(size 0.8)
 		(drill 0.4)
@@
 	)
 	(via
-		(at 49.119999 91.5)
+		(at 49.119999 91.4)
 		(size 0.8)
 		(drill 0.4)
@@
 	)
 	(via
-		(at 66.899999 91.5)
+		(at 66.899999 91.4)
 		(size 0.8)
 		(drill 0.4)
@@
 	)
 	(via
-		(at 51.659999 93.5)
+		(at 51.659999 93.6)
 		(size 0.8)
 		(drill 0.4)
@@
 	)
 	(via
-		(at 71.979999 91.5)
+		(at 71.979999 91.4)
 		(size 0.8)
 		(drill 0.4)
@@
 	)
 	(via
-		(at 69.439999 91.5)
+		(at 69.439999 91.4)
 		(size 0.8)
 		(drill 0.4)
@@
 	)
 	(via
-		(at 69.439999 93.5)
+		(at 69.439999 93.6)
 		(size 0.8)
 		(drill 0.4)
@@
 	)
 	(via
-		(at 41.499999 93.5)
+		(at 41.499999 93.6)
 		(size 0.8)
 		(drill 0.4)
@@
 	)
 	(via
-		(at 56.739999 93.5)
+		(at 56.739999 93.6)
 		(size 0.8)
 		(drill 0.4)
@@
 	)
 	(via
-		(at 56.739999 91.5)
+		(at 56.739999 91.4)
 		(size 0.8)
 		(drill 0.4)
@@
 	)
 	(via
-		(at 71.979999 93.5)
+		(at 71.979999 93.6)
 		(size 0.8)
 		(drill 0.4)
@@
 	)
 	(via
-		(at 44.039999 91.5)
+		(at 44.039999 91.4)
 		(size 0.8)
 		(drill 0.4)
@@
 	)
 	(via
-		(at 44.039999 93.5)
+		(at 44.039999 93.6)
 		(size 0.8)
 		(drill 0.4)
@@
 	)
 	(via
-		(at 54.199999 91.5)
+		(at 54.199999 91.4)
 		(size 0.8)
 		(drill 0.4)
@@
 	)
 	(via
-		(at 41.499999 91.5)
+		(at 41.499999 91.4)
 		(size 0.8)
 		(drill 0.4)
@@
 	)
 	(via
-		(at 64.359999 93.5)
+		(at 64.359999 93.6)
 		(size 0.8)
 		(drill 0.4)
@@
 	)
 	(via
-		(at 49.119999 93.5)
+		(at 49.119999 93.6)
 		(size 0.8)
 		(drill 0.4)
@@
 	)
 	(via
-		(at 77.059999 91.5)
+		(at 77.059999 91.4)
 		(size 0.8)
 		(drill 0.4)
@@
 	)
 	(via
-		(at 74.519999 91.5)
+		(at 74.519999 91.4)
 		(size 0.8)
 		(drill 0.4)
@@
 	)
 	(segment
-		(start 35.75 86.2)
-		(end 36.419999 86.869999)
+		(start 35.15 84.1)
+		(end 35.75 84.7)
 		(width 0.25)
 		(layer "F.Cu")
@@
 	)
 	(segment
-		(start 35.75 85)
-		(end 35.75 86.2)
+		(start 35.15 83.84)
+		(end 35.15 84.1)
 		(width 0.25)
 		(layer "F.Cu")
@@
 	)
 	(segment
-		(start 36.419999 86.869999)
-		(end 36.419999 88.630001)
+		(start 35.75 86.2)
+		(end 36.419999 86.869999)
 		(width 0.25)
 		(layer "F.Cu")
@@
 	)
 	(segment
-		(start 35.15 84.4)
-		(end 35.75 85)
+		(start 36.419999 88.630001)
+		(end 35.15 89.9)
 		(width 0.25)
 		(layer "F.Cu")
@@
 	)
 	(segment
-		(start 35.15 83.84)
-		(end 35.15 84.4)
+		(start 36.419999 86.869999)
+		(end 36.419999 88.630001)
 		(width 0.25)
 		(layer "F.Cu")
@@
 	)
 	(segment
-		(start 36.419999 88.630001)
-		(end 35.15 89.9)
+		(start 35.75 84.7)
+		(end 35.75 86.2)
 		(width 0.25)
 		(layer "F.Cu")

Commit message: updated connector yet again (previous versions will not work)
Routing:
- net GND: track 92.9 -> 134.8 mm, vias 135 -> 123
- net +3.3V: track 149.8 -> 170.8 mm
- net +5V: track 152.2 -> 132.3 mm, vias 0 -> 1
- net Net-(J1-~{CE0}_SPI0/GPIO08): track 7.12 -> 3.52 mm
- net Net-(J1-GPIO18/SPI1_~{CE0}/PCM_CLK/PWM0): track 7.11 -> 3.52 mm
- net Net-(J1-GPIO20/SPI1_MOSI/PCM_DIN/PWM1): track 7.11 -> 3.52 mm
- net Net-(J1-GPIO16/SPI1_~{CE2}): track 7.11 -> 3.52 mm
- net Net-(J1-~{CE1}_SPI0/GPIO07): track 7.11 -> 3.52 mm
- net Net-(J1-ID_SC_I2C0/GPIO01): track 7.11 -> 3.52 mm
- net Net-(J1-GPIO25/SDIO_DAT1): track 7.11 -> 3.52 mm
- net Net-(J1-GPIO24/SDIO_DAT0): track 7.11 -> 3.52 mm
- net Net-(J1-GPIO23/SDIO_CMD): track 7.11 -> 3.52 mm
- net Net-(J1-GPIO14/UART_TXD): track 14.1 -> 10.5 mm, vias 0 -> 1
- net Net-(J1-GPIO12/PWM0): track 15.1 -> 11.5 mm, vias 0 -> 1
- net Net-(J1-GPIO15/UART_RXD): track 14.4 -> 10.8 mm, vias 0 -> 1
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- added copper zone on B.Cu, net +5V

Commit message: pcb version bump
Routing:
- net +3.3V: track 170.8 -> 172.4 mm
- net GND: vias 123 -> 125
Other:
- board text added: "${TITLE} ${REVISION} 08/25 5V ONLY FANS"
- board text removed: "${TITLE} ${REVISION} 02/25 5V ONLY FANS"
